File: Schematics/65C02_Computer/6502_IO.sch (KiCad schematic (older format))
At the start: 30 parts, among them J10 VIA2PB, J11 LCD Connector, J2 Optional UART Port, J3 USB_B_Micro, J4 USB_B, J5 Power Connector, J6 Mini-DIN-6, J8 AVR-ISP-10, J9 VIA2PA, U10 ATtiny4313-PU, U11 65C22S, U12 65C22S, U5 65C51N, U6 FT230XS, X2 1.8432MHz

Commit message: Updated schematics and board files to V002
Parts:
- removed J11: LCD Connector, Connector_PinSocket_2.54mm:PinSocket_1x16_P2.54mm_Vertical, symbol Connector:Conn_01x16_Female
- removed J3: USB_B_Micro, Connector_USB:USB_Micro-B_Molex-105017-0001, symbol Connector:USB_B_Micro
- removed J4: USB_B, Connector_USB:USB_B_OST_USB-B1HSxx_Horizontal, symbol 6502:USB_B
- removed J6: Mini-DIN-6, 65C02_Computer:mini_din-6, symbol Connector:Mini-DIN-6
- removed J8: AVR-ISP-10, Connector_PinHeader_2.54mm:PinHeader_2x03_P2.54mm_Vertical, symbol Connector:AVR-ISP-6
- removed U10: ATtiny4313-PU, Package_DIP:DIP-20_W7.62mm_Socket, symbol MCU_Microchip_ATtiny:ATtiny4313-PU
- added J12: VIA1PA, Connector_PinSocket_2.54mm:PinSocket_1x12_P2.54mm_Vertical, symbol Connector:Conn_01x12_Male
- added J13: VIA1PB, Connector_PinSocket_2.54mm:PinSocket_1x12_P2.54mm_Vertical, symbol Connector:Conn_01x12_Male
- added J14: LCD Connector, 65C02_Computer:LCD-4line, symbol Connector:Conn_01x16_Female
- added J15: LCD Support, Connector_PinSocket_2.54mm:PinSocket_1x16_P2.54mm_Vertical, symbol Connector:Conn_01x16_Female
- added J2: USB_B_Mini, Connectors:USB-MINI-B-PTH-1734510, symbol 6502:USB_B_Mini
- added J42, J43, J44, J45, J47, J48, J49, J50, J51, J60, J61, J62, J63, J64: Jumper_NC_Small, 65C02_Computer:PinHeader_1x02_P2.54mm_Vertical_Close, symbol Device:Jumper_NC_Small
- added J46: Jumper_NC_Small, Connector_PinHeader_2.54mm:PinHeader_1x02_P2.54mm_Vertical, symbol Device:Jumper_NC_Small
- added J53, J54, J55, J56, J57, J58, J59: Jumper_3_Bridged12, 65C02_Computer:PinHeader_1x03_P2.54mm_Vertical_Close, symbol Jumper:Jumper_3_Bridged12
- J1: renamed from J2; footprint Connector_PinSocket_2.54mm:PinSocket_1x06_P2.54mm_Vertical -> 65C02_Computer:PinSocket_1x06_P2.54mm_Horizontal
- J10: renamed from J9; footprint Connector_PinHeader_2.54mm:PinHeader_1x12_P2.54mm_Vertical -> Connector_PinSocket_2.54mm:PinSocket_1x12_P2.54mm_Vertical
- J11: renamed from J10; footprint Connector_PinHeader_2.54mm:PinHeader_1x12_P2.54mm_Vertical -> Connector_PinSocket_2.54mm:PinSocket_1x12_P2.54mm_Vertical
- RV1: footprint Potentiometer_THT:Potentiometer_Piher_PT-10-V10_Vertical -> Potentiometer_THT:Potentiometer_Piher_PT-6-V_Vertical
- renumbered D4 to D1, D3 to D2, D2 to D3, D1 to D4, J5 to J3, U11 to U12, U12 to U13
Connections:
- net labels added: e, lcd0, lcd1, lcd2, lcd3, lcd4, lcd5, lcd6, lcd7, rs, rw, v1pa[0..9], v1pb8, v1pb9, v1pb[0..9], v2pa[0..9], v2pb[0..9]
- net labels removed: KBCLK, KBDAT
- wire segments 296 -> 342
- no-connect marks 17 -> 22
Other:
- note added: "ACIA 8200-820F"
- note added: "DB6502 2>3"
- note added: "Jumpers"
- note added: "KrisOS 1>2"
- note added: "LCD"
- note added: "VIA 1 9000-900F"
- note added: "VIA2 8800-880F"
- moved on the sheet: C10, C8, C9, D1, D2, D3, D4, FB1, J1, J10, J11, J3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
