File: Schematics/65C02_Computer/65C02_Computer.sch (KiCad schematic (older format))
At the start: 32 parts, among them J1 CLK Jumper, J7 Expansion port, SW1 RESET, U1 74HC21, U2 74HC00, U3 74HC02, U4 NE555, U7 65C02S, U8 28C256, U9 62256, X1 1MHz

Commit message: Updated schematics and board files to V002
Parts:
- removed J1: CLK Jumper, Connector_PinHeader_2.54mm:PinHeader_1x03_P2.54mm_Vertical, symbol Connector:Conn_01x03_Male
- removed R13: 4K7, Resistor_THT:R_Axial_DIN0207_L6.3mm_D2.5mm_P7.62mm_Horizontal, symbol Device:R
- added C18, C20, C21, C22, C23: 0.1uF, Capacitor_THT:C_Disc_D3.4mm_W2.1mm_P2.50mm, symbol Device:C
- added H1, H3, H4, H5, H6, H7: 3mm_MountingHole_Pad, 65C02_Computer:MountingHole_3.2mm_Pad, symbol Mechanical:MountingHole_Pad
- added H2: 3m_MountingHole_Pad, 65C02_Computer:MountingHole_3.2mm_Pad, symbol Mechanical:MountingHole_Pad
- added J16, J17, J22, J23, J35, J39, J40, J41: J, 65C02_Computer:PinHeader_1x02_P2.54mm_Vertical_Close, symbol Device:Jumper_NC_Small
- added J18, J36, J37: J, 65C02_Computer:PinHeader_1x02_P2.54mm_Vertical_Close, symbol Device:Jumper_NO_Small
- added J19, J20, J21, J24, J25, J27, J28, J30, J31, J33, J34: Jumper_NC_Small, 65C02_Computer:PinHeader_1x02_P2.54mm_Vertical_Close, symbol Device:Jumper_NC_Small
- added J26, J29, J32: Conn_01x01, 65C02_Computer:PinHeader_1x01_P2.54mm_Vertical_Close, symbol Connector_Generic:Conn_01x01
- added LOGO1: Logo_Open_Hardware_Small, Symbol:KiCad-Logo2_5mm_SilkScreen, symbol Graphic:Logo_Open_Hardware_Small
- added LOGO2: Logo_Open_Hardware_Small, Symbol:OSHW-Logo_5.7x6mm_SilkScreen, symbol Graphic:Logo_Open_Hardware_Small
- added R14, R15, R17: 4K7, Resistor_THT:R_Axial_DIN0207_L6.3mm_D2.5mm_P7.62mm_Horizontal, symbol Device:R
Connections:
- net +5V: now also C18.1, C20.1, C21.1, C22.1, C23.1, J19.2, R14.1, R15.1, R17.1; no longer U7.36 (BE), U7.38 (~SO), U8.27 (~WE)
- net CLK: now also J35.2, J36.2, J37.2
- net CLKOUT: now also J35.1
- net GND: now also C18.2, C20.2, C21.2, C22.2, C23.2, J24.1, J25.1, J27.1, J28.1, J30.1, J31.1, J37.1; no longer U1.10, U1.12, U1.13, U1.9, U3.11, U3.12, U3.5, U3.6, U3.8, U3.9
- net ~IRQX: now also U1.10, J39.2; no longer U1.5
- net ~RAM_CS: now also J33.2, J34.2; no longer U9.20 (~CE), U9.22 (~OE)
- net ~ROM_CS: now also J21.2; no longer U8.20 (~CE)
- net ~ROM_OE: now also J20.2; no longer U8.22 (~OE)
- net at R7.1: now also J16.1; no longer U7.2 (RDY)
- net at R8.1: now also J17.1; no longer U7.6 (~NMI)
- net sync: now reaches U7.7 (SYNC)
- net sync: now also J18.2
- net at U1.8: now also U1.5
- net at U3.4: now also J26.1 (Pin_1)
- net at U3.10: now also J29.1 (Pin_1)
- net at U3.13: now also J32.1 (Pin_1)
- new net: J34.1, U9.20 (~CE)
- new net: J33.1, U9.22 (~OE)
- new net: J21.1, U8.20 (~CE)
- new net: J20.1, U8.22 (~OE)
- new net: J19.1, U8.27 (~WE)
- new net: J40.2, U1.12
- new net: J41.2, U1.13
- new net: J25.2, U3.5
- new net: J24.2, U3.6
- new net: J27.2, U3.8
- new net: J28.2, U3.9
- new net: J30.2, U3.11
- new net: J31.2, U3.12
- new net: J39.1, J40.1, J41.1, R17.2
- new net: J22.2, R14.2
- new net: J23.2, R15.2
- new net 4Mhz_CLK: J36.1
- new net be: J23.1, U7.36 (BE)
- new net rdy: J16.2, U7.2 (RDY)
- new net ~V3IRQ: U1.9
- new net ~nmi: J17.2, U7.6 (~NMI)
- new net ~so: J22.1, U7.38 (~SO)
- no-connect marks 11 -> 14
Other:
- note added: "External CLK"
- note added: "RAM 32K 0000-7FFF"
- note added: "ROM 24K A000-FFFF"
- note added: "^"
- moved on the sheet: C1, C11, C12, C13, C14, C15, C16, C17, C2, C3, C7, R7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

Commit message: Update files to v002
Parts:
- removed J35: J, 65C02_Computer:PinHeader_1x02_P2.54mm_Vertical_Close, symbol Device:Jumper_NC_Small
- removed J36, J37: J, 65C02_Computer:PinHeader_1x02_P2.54mm_Vertical_Close, symbol Device:Jumper_NO_Small
- added J35: CLK Jumper, 65C02_Computer:PinHeader_1x03_P2.54mm_Vertical_Close, symbol Connector:Conn_01x03_Male
Connections:
- net CLK: now also J35.2 (Pin_2)
- net CLKOUT: now also J35.1 (Pin_1)
- net GND: now also J35.3 (Pin_3)
Other:
- note removed: "External CLK"
- note removed: "^"
Changed lines of the file:
@@
 Sheet 1 3
 Title "65C02 Hobby Computer"
-Date "2020-05-10"
+Date "2020-05-12"
 Rev "v002"
 Comp ""
@@
 Wire Wire Line
 	5700 6650 5850 6650
-$Comp
-L Device:Jumper_NC_Small J?
-U 1 1 5FB44899
-P 4400 2500
-AR Path="/5EA0A6F6/5FB44899" Ref="J?"  Part="1"
-AR Path="/5FB44899" Ref="J35"  Part="1"
-F 0 "J35" H 4410 2600 50  0000 C CNN
-F 1 "J" H 4400 2621 50  0001 C CNN
-F 2 "65C02_Computer:PinHeader_1x02_P2.54mm_Vertical_Close" H 4400 2500 50  0001 C CNN
-F 3 "~" H 4400 2500 50  0001 C CNN
-	1    4400 2500
-	1    0    0    -1
-$EndComp
-$Comp
-L Device:Jumper_NO_Small J?
-U 1 1 5FB46024
-P 4400 2650
-AR Path="/5EA0A6F6/5FB46024" Ref="J?"  Part="1"
-AR Path="/5FB46024" Ref="J36"  Part="1"
-F 0 "J36" H 4410 2720 50  0000 C CNN
-F 1 "J" H 4400 2744 50  0001 C CNN
-F 2 "65C02_Computer:PinHeader_1x02_P2.54mm_Vertical_Close" H 4400 2650 50  0001 C CNN
-F 3 "~" H 4400 2650 50  0001 C CNN
-	1    4400 2650
-	1    0    0    -1
-$EndComp
-$Comp
-L Device:Jumper_NO_Small J?
-U 1 1 5FB6B847
-P 4400 2800
-AR Path="/5EA0A6F6/5FB6B847" Ref="J?"  Part="1"
-AR Path="/5FB6B847" Ref="J37"  Part="1"
-F 0 "J37" H 4390 2870 50  0000 C CNN
-F 1 "J" H 4400 2894 50  0001 C CNN
-F 2 "65C02_Computer:PinHeader_1x02_P2.54mm_Vertical_Close" H 4400 2800 50  0001 C CNN
-F 3 "~" H 4400 2800 50  0001 C CNN
-	1    4400 2800
-	1    0    0    -1
-$EndComp
-Wire Wire Line
-	4500 2500 4550 2500
-Wire Wire Line
-	4550 2500 4550 2650
-Wire Wire Line
-	4550 2800 4500 2800
-Wire Wire Line
-	4500 2650 4550 2650
-Connection ~ 4550 2650
-Wire Wire Line
-	4550 2650 4550 2800
-Text GLabel 4650 2650 2    50   Output ~ 0
+Text GLabel 4250 2650 0    50   Output ~ 0
 CLK
-Wire Wire Line
-	4550 2650 4650 2650
-Text GLabel 4200 2500 0    50   Input ~ 0
+Text GLabel 4250 2550 0    50   Input ~ 0
 CLKOUT
-Text GLabel 4200 2650 0    50   Input ~ 0
-4Mhz_CLK
-Wire Wire Line
-	4200 2500 4300 2500
-Wire Wire Line
-	4300 2650 4200 2650
-Wire Wire Line
-	4200 2800 4300 2800
-Text Notes 4200 2950 0    50   ~ 0
-External CLK
-Text GLabel 4200 2800 0    50   Input ~ 0
+Wire Wire Line
+	4250 2550 4350 2550
+Wire Wire Line
+	4350 2650 4250 2650
+Text GLabel 4250 2750 0    50   Input ~ 0
 GND
-Text Notes 4340 3070 0    197  ~ 0
-^
 $Comp
 L Oscillator:ACO-xxxMHz X1
@@
 Wire Wire Line
 	10400 3750 9950 3750
+$Comp
+L Connector:Conn_01x03_Male J35
+U 1 1 5EC51313
+P 4550 2650
+F 0 "J35" H 4522 2674 50  0000 R CNN
+F 1 "CLK Jumper" H 4522 2583 50  0000 R CNN
+F 2 "65C02_Computer:PinHeader_1x03_P2.54mm_Vertical_Close" H 4550 2650 50  0001 C CNN
+F 3 "~" H 4550 2650 50  0001 C CNN
+	1    4550 2650
+	-1   0    0    -1
+$EndComp
+Wire Wire Line
+	4350 2750 4250 2750
 Wire Bus Line
 	3100 5450 3100 5650
