File: Schematics/65C02_Computer/65C02_Computer.kicad_pcb (KiCad board)
At the start: 2 copper layers, 203.2 x 149.9 mm, 68 parts, among them J1 CLK Jumper, J10 VIA2PB, J11 LCD Connector, J2 Optional UART Port, J3 USB_B_Micro, J4 USB_B, J5 Power Connector, J6 Mini-DIN-6, J7 Expansion port, J8 AVR-ISP-10, J9 VIA2PA, SW1 RESET, U1 74HC21, U10 ATtiny4313-PU, U11 65C22S, U12 65C22S, U2 74HC00, U3 74HC02, U4 NE555, U5 65C51N, U6 FT230XS, U7 65C02S, U8 28C256, U9 62256, X1 1MHz, X2 1.8432MHz

Commit message: Updated schematics and board files to V002
Parts:
- removed the J3 at (218.3, 39.4)
- removed the J4 at (205.7, 59.7)
- removed R13: 4K7, Resistor_THT:R_Axial_DIN0207_L6.3mm_D2.5mm_P7.62mm_Horizontal
- removed REF**: KiCad-Logo2_8mm_SilkScreen, Symbol:KiCad-Logo2_8mm_SilkScreen
- removed REF**: OSHW-Logo_11.4x12mm_SilkScreen, Symbol:OSHW-Logo_11.4x12mm_SilkScreen
- removed REF** (x4): MountingHole_3mm_Pad, MountingHole:MountingHole_3mm_Pad
- added C18: 0.1uF, Capacitor_THT:C_Disc_D3.4mm_W2.1mm_P2.50mm, F.Cu at (69.8, 149.9)
- added C19: 1uf, Capacitor_THT:C_Disc_D3.4mm_W2.1mm_P2.50mm, F.Cu at (212.7, 113.7)
- added C20: 0.1uF, Capacitor_THT:C_Disc_D3.4mm_W2.1mm_P2.50mm, F.Cu at (212.7, 118.7)
- added C21: 0.1uF, Capacitor_THT:C_Disc_D3.4mm_W2.1mm_P2.50mm, F.Cu at (27.9, 73.0)
- added C22: 0.1uF, Capacitor_THT:C_Disc_D3.4mm_W2.1mm_P2.50mm, F.Cu at (144.1, 63.5)
- added C23: 0.1uF, Capacitor_THT:C_Disc_D3.4mm_W2.1mm_P2.50mm, F.Cu at (192.4, 148.6)
- added H1: 3mm_MountingHole_Pad, 65C02_Computer:MountingHole_3.2mm_Pad, F.Cu at (24.1, 26.7)
- added H2: 3m_MountingHole_Pad, 65C02_Computer:MountingHole_3.2mm_Pad, F.Cu at (214.6, 26.7)
- added H3: 3mm_MountingHole_Pad, 65C02_Computer:MountingHole_3.2mm_Pad, F.Cu at (214.6, 163.8)
- added H4: 3mm_MountingHole_Pad, 65C02_Computer:MountingHole_3.2mm_Pad, F.Cu at (24.1, 163.8)
- added H5: 3mm_MountingHole_Pad, 65C02_Computer:MountingHole_3.2mm_Pad, F.Cu at (24.1, 77.5)
- added H6: 3mm_MountingHole_Pad, 65C02_Computer:MountingHole_3.2mm_Pad, F.Cu at (74.3, 163.8)
- added H7: 3mm_MountingHole_Pad, 65C02_Computer:MountingHole_3.2mm_Pad, F.Cu at (128.9, 163.8)
- added J12: VIA1PA, Connector_PinSocket_2.54mm:PinSocket_1x12_P2.54mm_Vertical, F.Cu at (141.0, 157.5)
- added J13: VIA1PB, Connector_PinSocket_2.54mm:PinSocket_1x12_P2.54mm_Vertical, F.Cu at (141.0, 165.1)
- added J14: LCD Connector, 65C02_Computer:LCD-4line, F.Cu at (106.7, 69.8)
- added J15: LCD Support, Connector_PinSocket_2.54mm:PinSocket_1x16_P2.54mm_Vertical, F.Cu at (106.7, 95.2)
- added J16: J, 65C02_Computer:PinHeader_1x02_P2.54mm_Vertical_Close, F.Cu at (43.2, 75.6)
- added J17: J, 65C02_Computer:PinHeader_1x02_P2.54mm_Vertical_Close, F.Cu at (53.3, 75.6)
- added J18: J, 65C02_Computer:PinHeader_1x02_P2.54mm_Vertical_Close, F.Cu at (58.4, 75.6)
- added J19: Jumper_NC_Small, 65C02_Computer:PinHeader_1x02_P2.54mm_Vertical_Close, F.Cu at (59.1, 83.2)
- added J20: Jumper_NC_Small, 65C02_Computer:PinHeader_1x02_P2.54mm_Vertical_Close, F.Cu at (59.1, 86.4)
- added J21: Jumper_NC_Small, 65C02_Computer:PinHeader_1x02_P2.54mm_Vertical_Close, F.Cu at (59.1, 89.5)
- added J22: J, 65C02_Computer:PinHeader_1x02_P2.54mm_Vertical_Close, F.Cu at (45.7, 49.5)
- added J23: J, 65C02_Computer:PinHeader_1x02_P2.54mm_Vertical_Close, F.Cu at (52.7, 49.5)
- added J24: Jumper_NC_Small, 65C02_Computer:PinHeader_1x02_P2.54mm_Vertical_Close, F.Cu at (73.7, 35.6)
- added J25: Jumper_NC_Small, 65C02_Computer:PinHeader_1x02_P2.54mm_Vertical_Close, F.Cu at (73.7, 33.0)
- added J26: Conn_01x01, 65C02_Computer:PinHeader_1x01_P2.54mm_Vertical_Close, F.Cu at (76.2, 30.5)
- added J27: Jumper_NC_Small, 65C02_Computer:PinHeader_1x02_P2.54mm_Vertical_Close, F.Cu at (73.7, 43.2)
- added J28: Jumper_NC_Small, 65C02_Computer:PinHeader_1x02_P2.54mm_Vertical_Close, F.Cu at (73.7, 40.6)
- added J29: Conn_01x01, 65C02_Computer:PinHeader_1x01_P2.54mm_Vertical_Close, F.Cu at (76.2, 38.1)
- added J30: Jumper_NC_Small, 65C02_Computer:PinHeader_1x02_P2.54mm_Vertical_Close, F.Cu at (73.7, 27.9)
- added J31: Jumper_NC_Small, 65C02_Computer:PinHeader_1x02_P2.54mm_Vertical_Close, F.Cu at (73.7, 25.4)
- added J32: Conn_01x01, 65C02_Computer:PinHeader_1x01_P2.54mm_Vertical_Close, F.Cu at (76.2, 22.9)
- added J33: Jumper_NC_Small, 65C02_Computer:PinHeader_1x02_P2.54mm_Vertical_Close, F.Cu at (85.7, 81.3)
- added J34: Jumper_NC_Small, 65C02_Computer:PinHeader_1x02_P2.54mm_Vertical_Close, F.Cu at (85.7, 84.5)
- added J35: J, 65C02_Computer:PinHeader_1x02_P2.54mm_Vertical_Close, F.Cu at (30.5, 38.1)
- added J36: J, 65C02_Computer:PinHeader_1x02_P2.54mm_Vertical_Close, F.Cu at (30.5, 40.6)
- added J37: J, 65C02_Computer:PinHeader_1x02_P2.54mm_Vertical_Close, F.Cu at (30.5, 43.2)
- added J39: J, 65C02_Computer:PinHeader_1x02_P2.54mm_Vertical_Close, F.Cu at (30.5, 29.2)
- added J40: J, 65C02_Computer:PinHeader_1x02_P2.54mm_Vertical_Close, F.Cu at (30.5, 31.8)
- added J41: J, 65C02_Computer:PinHeader_1x02_P2.54mm_Vertical_Close, F.Cu at (30.5, 34.3)
- added J42: Jumper_NC_Small, 65C02_Computer:PinHeader_1x02_P2.54mm_Vertical_Close, F.Cu at (186.1, 24.1)
- added J43: Jumper_NC_Small, 65C02_Computer:PinHeader_1x02_P2.54mm_Vertical_Close, F.Cu at (176.5, 155.6)
- added J44: Jumper_NC_Small, 65C02_Computer:PinHeader_1x02_P2.54mm_Vertical_Close, F.Cu at (176.5, 153.0)
- added J45: Jumper_NC_Small, 65C02_Computer:PinHeader_1x02_P2.54mm_Vertical_Close, F.Cu at (193.7, 24.1)
- added J46: Jumper_NC_Small, Connector_PinHeader_2.54mm:PinHeader_1x02_P2.54mm_Vertical, F.Cu at (138.4, 24.1)
- added J47: Jumper_NC_Small, 65C02_Computer:PinHeader_1x02_P2.54mm_Vertical_Close, F.Cu at (179.7, 36.8)
- added J48: Jumper_NC_Small, 65C02_Computer:PinHeader_1x02_P2.54mm_Vertical_Close, F.Cu at (179.7, 34.3)
- added J49: Jumper_NC_Small, 65C02_Computer:PinHeader_1x02_P2.54mm_Vertical_Close, F.Cu at (121.9, 155.6)
- added J5: AudioJack SJ1-3523N, 65C02_Computer:Jack_3.5mm_CUI_SJ1-3523N_Horizontal, F.Cu at (212.5, 102.8)
- added J50: Jumper_NC_Small, 65C02_Computer:PinHeader_1x02_P2.54mm_Vertical_Close, F.Cu at (121.9, 153.0)
- added J51: Jumper_NC_Small, 65C02_Computer:PinHeader_1x02_P2.54mm_Vertical_Close, F.Cu at (163.2, 53.3)
- added J53: Jumper_3_Bridged12, 65C02_Computer:PinHeader_1x03_P2.54mm_Vertical_Close, F.Cu at (114.3, 56.5)
- added J54: Jumper_3_Bridged12, 65C02_Computer:PinHeader_1x03_P2.54mm_Vertical_Close, F.Cu at (116.8, 56.5)
- added J55: Jumper_3_Bridged12, 65C02_Computer:PinHeader_1x03_P2.54mm_Vertical_Close, F.Cu at (119.4, 56.5)
- added J56: Jumper_3_Bridged12, 65C02_Computer:PinHeader_1x03_P2.54mm_Vertical_Close, F.Cu at (121.9, 56.5)
- added J57: Jumper_3_Bridged12, 65C02_Computer:PinHeader_1x03_P2.54mm_Vertical_Close, F.Cu at (124.5, 56.5)
- added J58: Jumper_3_Bridged12, 65C02_Computer:PinHeader_1x03_P2.54mm_Vertical_Close, F.Cu at (127.0, 56.5)
- added J59: Jumper_3_Bridged12, 65C02_Computer:PinHeader_1x03_P2.54mm_Vertical_Close, F.Cu at (129.5, 56.5)
- added J60: Jumper_NC_Small, 65C02_Computer:PinHeader_1x02_P2.54mm_Vertical_Close, F.Cu at (132.1, 57.8)
- added J61: Jumper_NC_Small, 65C02_Computer:PinHeader_1x02_P2.54mm_Vertical_Close, F.Cu at (134.6, 57.8)
- added J62: Jumper_NC_Small, 65C02_Computer:PinHeader_1x02_P2.54mm_Vertical_Close, F.Cu at (137.2, 57.8)
- added J63: Jumper_NC_Small, 65C02_Computer:PinHeader_1x02_P2.54mm_Vertical_Close, F.Cu at (139.7, 57.8)
- added J64: Jumper_NC_Small, 65C02_Computer:PinHeader_1x02_P2.54mm_Vertical_Close, F.Cu at (206.4, 24.1)
- added J65: Jumper_NC_Small, 65C02_Computer:PinHeader_1x02_P2.54mm_Vertical_Close, F.Cu at (67.3, 155.6)
- added J66: Jumper_NC_Small, 65C02_Computer:PinHeader_1x02_P2.54mm_Vertical_Close, F.Cu at (67.3, 153.0)
- added J67: Jumper_NC_Small, 65C02_Computer:PinHeader_1x02_P2.54mm_Vertical_Close, F.Cu at (186.7, 72.4)
- added J68: Jumper_NC_Small, 65C02_Computer:PinHeader_1x02_P2.54mm_Vertical_Close, F.Cu at (186.7, 74.9)
- added J69: Jumper_NC_Small, 65C02_Computer:PinHeader_1x02_P2.54mm_Vertical_Close, F.Cu at (186.7, 77.5)
- added J70: Jumper_NC_Small, 65C02_Computer:PinHeader_1x02_P2.54mm_Vertical_Close, F.Cu at (186.7, 80.0)
- added J71: Jumper_NC_Small, 65C02_Computer:PinHeader_1x02_P2.54mm_Vertical_Close, F.Cu at (186.7, 82.5)
- added J72: Jumper_NC_Small, 65C02_Computer:PinHeader_1x02_P2.54mm_Vertical_Close, F.Cu at (186.7, 85.1)
- added J73: Jumper_NC_Small, 65C02_Computer:PinHeader_1x02_P2.54mm_Vertical_Close, F.Cu at (186.7, 87.6)
- added J74: Jumper_NC_Small, 65C02_Computer:PinHeader_1x02_P2.54mm_Vertical_Close, F.Cu at (186.7, 90.2)
- added J75: Jumper_NC_Small, 65C02_Computer:PinHeader_1x02_P2.54mm_Vertical_Close, F.Cu at (186.7, 92.7)
- added J76: Jumper_NC_Small, 65C02_Computer:PinHeader_1x02_P2.54mm_Vertical_Close, F.Cu at (186.7, 95.2)
- added J77: Jumper_NC_Small, 65C02_Computer:PinHeader_1x02_P2.54mm_Vertical_Close, F.Cu at (186.7, 97.8)
- added J78: Jumper_NC_Small, 65C02_Computer:PinHeader_1x02_P2.54mm_Vertical_Close, F.Cu at (186.7, 100.3)
- added J79: Conn_01x01, 65C02_Computer:PinHeader_1x01_P2.54mm_Vertical_Close, F.Cu at (186.7, 102.9)
- added J8: VIA3PA, Connector_PinSocket_2.54mm:PinSocket_1x12_P2.54mm_Vertical, F.Cu at (31.8, 157.5)
- added J80: Conn_01x01, 65C02_Computer:PinHeader_1x01_P2.54mm_Vertical_Close, F.Cu at (186.7, 105.4)
- added J81: Conn_01x01, 65C02_Computer:PinHeader_1x01_P2.54mm_Vertical_Close, F.Cu at (186.7, 108.0)
- added J82: Jumper_NC_Small, 65C02_Computer:PinHeader_1x02_P2.54mm_Vertical_Close, F.Cu at (196.8, 120.0)
- added J83: Jumper_NC_Small, 65C02_Computer:PinHeader_1x02_P2.54mm_Vertical_Close, F.Cu at (196.8, 122.6)
- added J84: Jumper_NC_Small, 65C02_Computer:PinHeader_1x02_P2.54mm_Vertical_Close, F.Cu at (196.8, 125.1)
- added J85: Jumper_NC_Small, 65C02_Computer:PinHeader_1x02_P2.54mm_Vertical_Close, F.Cu at (196.8, 127.6)
- added J86: Jumper_NC_Small, 65C02_Computer:PinHeader_1x02_P2.54mm_Vertical_Close, F.Cu at (196.8, 130.2)
- added J87: Jumper_NC_Small, 65C02_Computer:PinHeader_1x02_P2.54mm_Vertical_Close, F.Cu at (196.8, 132.7)
- added J88: Jumper_NC_Small, 65C02_Computer:PinHeader_1x02_P2.54mm_Vertical_Close, F.Cu at (196.8, 135.3)
- added J89: Jumper_NC_Small, 65C02_Computer:PinHeader_1x02_P2.54mm_Vertical_Close, F.Cu at (196.8, 137.8)
- added J90: Jumper_NC_Small, 65C02_Computer:PinHeader_1x02_P2.54mm_Vertical_Close, F.Cu at (196.8, 140.3)
- added J91: Jumper_NC_Small, 65C02_Computer:PinHeader_1x02_P2.54mm_Vertical_Close, F.Cu at (196.8, 142.9)
- added J92: Jumper_NO_Small, 65C02_Computer:PinHeader_1x02_P2.54mm_Vertical_Close, F.Cu at (195.6, 165.1)
- added LOGO1: Logo_Open_Hardware_Small, Symbol:KiCad-Logo2_5mm_SilkScreen, B.Cu at (162.6, 104.8)
- added LOGO2: Logo_Open_Hardware_Small, Symbol:OSHW-Logo_5.7x6mm_SilkScreen, B.Cu at (163.2, 114.3)
- added R14: 4K7, Resistor_THT:R_Axial_DIN0207_L6.3mm_D2.5mm_P7.62mm_Horizontal, F.Cu at (31.8, 47.6)
- added R15: 4K7, Resistor_THT:R_Axial_DIN0207_L6.3mm_D2.5mm_P7.62mm_Horizontal, F.Cu at (64.8, 48.3)
- added R16: 1K, Resistor_THT:R_Axial_DIN0207_L6.3mm_D2.5mm_P7.62mm_Horizontal, F.Cu at (201.3, 113.7)
- added R17: 4K7, Resistor_THT:R_Axial_DIN0207_L6.3mm_D2.5mm_P7.62mm_Horizontal, F.Cu at (36.2, 25.4)
- added U13: 65C22S, Package_DIP:DIP-40_W15.24mm_Socket, F.Cu at (130.8, 146.1)
- added U14: SN76489AN, Package_DIP:DIP-16_W7.62mm_Socket, F.Cu at (206.4, 122.6)
- added X3: 4 MHz, Oscillator:Oscillator_DIP-14, F.Cu at (197.5, 156.2)
- D1: value PWR -> BLINK
- D2: value TX -> RX
- D3: value RX -> TX
- D4: value BLINK -> PWR
- J1: value CLK Jumper -> Optional UART Port; footprint Connector_PinHeader_2.54mm:PinHeader_1x03_P2.54mm_Vertical -> 65C02_Computer:PinSocket_1x06_P2.54mm_Horizontal
- J10: value VIA2PB -> VIA2PA; footprint Connector_PinHeader_2.54mm:PinHeader_1x12_P2.54mm_Vertical -> Connector_PinSocket_2.54mm:PinSocket_1x12_P2.54mm_Vertical
- J11: value LCD Connector -> VIA2PB; footprint Connector_PinSocket_2.54mm:PinSocket_1x16_P2.54mm_Vertical -> Connector_PinSocket_2.54mm:PinSocket_1x12_P2.54mm_Vertical
- J2: value Optional UART Port -> USB_B_Mini; footprint Connector_PinSocket_2.54mm:PinSocket_1x06_P2.54mm_Vertical -> Connectors:USB-MINI-B-PTH-1734510
- J9: value VIA2PA -> VIA3PB; footprint Connector_PinHeader_2.54mm:PinHeader_1x12_P2.54mm_Vertical -> Connector_PinSocket_2.54mm:PinSocket_1x12_P2.54mm_Vertical
- RV1: footprint Potentiometer_THT:Potentiometer_Piher_PT-10-V10_Vertical -> Potentiometer_THT:Potentiometer_Piher_PT-6-V_Vertical
- moved J1 179.9 mm to (210.2, 46.4), turned to 180 degrees
- moved J7 128.7 mm to (26.7, 83.8)
- moved RV1 112.8 mm to (97.2, 61.0)
- moved C16 95.3 mm to (179.1, 149.9), turned to 180 degrees
- moved C17 83.8 mm to (124.5, 149.9), turned to 180 degrees
- moved U12 78.9 mm to (76.2, 146.1)
- moved J11 78.8 mm to (86.4, 165.1)
- moved R3 67.0 mm to (58.4, 23.5), turned to 180 degrees
- moved J2 42.4 mm to (212.7, 55.2), turned to 90 degrees
- moved D1 30.5 mm to (163.8, 59.7)
- moved D4 30.5 mm to (194.3, 59.7)
- moved X2 22.2 mm to (156.2, 63.5), turned to 90 degrees
- moved R9 18.2 mm to (170.2, 55.9), turned to 270 degrees
- moved J10 17.3 mm to (86.4, 157.5)
- moved C15 10.9 mm to (201.9, 67.9), turned to 180 degrees
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- renumbered J5 to J3, J6 to J4, J8 to J6
Connections:
- J1 pad 1: GND -> ~RTS
- J1 pad 2: CLK -> TxD
- J1 pad 3: CLKOUT -> RxD
- J10 pad 1: /6502 Peripherals/v2pb0 -> v2pa0
- J10 pad 10: /6502 Peripherals/v2pb9 -> v2pa9
- J10 pad 2: /6502 Peripherals/v2pb1 -> v2pa1
- J10 pad 3: /6502 Peripherals/v2pb2 -> v2pa2
- J10 pad 4: /6502 Peripherals/v2pb3 -> v2pa3
- J10 pad 5: /6502 Peripherals/v2pb4 -> v2pa4
- J10 pad 6: /6502 Peripherals/v2pb5 -> v2pa5
- J10 pad 7: /6502 Peripherals/v2pb6 -> v2pa6
- J10 pad 8: /6502 Peripherals/v2pb7 -> v2pa7
- J10 pad 9: /6502 Peripherals/v2pb8 -> v2pa8
- J11 pad 1: GND -> v2pb0
- J11 pad 10: GND -> v2pb9
- J11 pad 11: /6502 Peripherals/v1pb4 -> GND
- J11 pad 12: /6502 Peripherals/v1pb5 -> +5V
- J11 pad 2: +5V -> v2pb1
- J11 pad 3: Net-(J11-Pad3) -> v2pb2
- J11 pad 4: /6502 Peripherals/v1pb1 -> v2pb3
- J11 pad 5: /6502 Peripherals/v1pb2 -> v2pb4
- J11 pad 6: /6502 Peripherals/v1pb3 -> v2pb5
- J11 pad 7: GND -> v2pb6
- J11 pad 8: GND -> v2pb7
- J11 pad 9: GND -> v2pb8
- J2 pad 1: TxD -> Net-(FB1-Pad2)
- J2 pad 2: RxD -> PUSBD-
- J2 pad 3: ~RTS -> PUSBD+
- J2 pad 4: ~CTS -> Net-(J2-Pad4)
- J6 pad 1: /6502 Peripherals/v1pa6 -> v1pa6
- J6 pad 3: /6502 Peripherals/v1pa7 -> v1pa7
- J6 pad 4: /6502 Peripherals/v1pa5 -> v1pa5
- J9 pad 1: /6502 Peripherals/v2pa0 -> /6502 Peripherals 1/v3pb0
- J9 pad 10: /6502 Peripherals/v2pa9 -> /6502 Peripherals 1/v3pb9
- J9 pad 2: /6502 Peripherals/v2pa1 -> /6502 Peripherals 1/v3pb1
- J9 pad 3: /6502 Peripherals/v2pa2 -> /6502 Peripherals 1/v3pb2
- J9 pad 4: /6502 Peripherals/v2pa3 -> /6502 Peripherals 1/v3pb3
- J9 pad 5: /6502 Peripherals/v2pa4 -> /6502 Peripherals 1/v3pb4
- J9 pad 6: /6502 Peripherals/v2pa5 -> /6502 Peripherals 1/v3pb5
- J9 pad 7: /6502 Peripherals/v2pa6 -> /6502 Peripherals 1/v3pb6
- J9 pad 8: /6502 Peripherals/v2pa7 -> /6502 Peripherals 1/v3pb7
- J9 pad 9: /6502 Peripherals/v2pa8 -> /6502 Peripherals 1/v3pb8
- R10 pad 2: Net-(D3-Pad2) -> Net-(D2-Pad2)
- R11 pad 2: Net-(D2-Pad2) -> Net-(D3-Pad2)
- R12 pad 2: Net-(D1-Pad2) -> Net-(D4-Pad2)
- R7 pad 1: Net-(R7-Pad1) -> Net-(J16-Pad1)
- R8 pad 1: Net-(R8-Pad1) -> Net-(J17-Pad1)
- R9 pad 1: /6502 Peripherals/v1pb0 -> Net-(J51-Pad2)
- R9 pad 2: Net-(D4-Pad2) -> Net-(D1-Pad2)
- RV1 pad 2: Net-(J11-Pad3) -> Net-(J14-Pad3)
- U1 pad 10: GND -> ~IRQX
- U1 pad 12: GND -> Net-(J40-Pad2)
- U1 pad 13: GND -> Net-(J41-Pad2)
- U1 pad 5: ~IRQX -> Net-(U1-Pad5)
- U1 pad 8: Net-(U1-Pad8) -> Net-(U1-Pad5)
- U1 pad 9: GND -> ~V3IRQ
- U10 pad 12: /6502 Peripherals/v1pa0 -> Net-(J67-Pad1)
- U10 pad 13: /6502 Peripherals/v1pa1 -> Net-(J68-Pad1)
- U10 pad 14: /6502 Peripherals/v1pa2 -> Net-(J69-Pad1)
- U10 pad 15: /6502 Peripherals/v1pa3 -> Net-(J70-Pad1)
- U10 pad 16: /6502 Peripherals/v1pa4 -> Net-(J71-Pad1)
- U10 pad 17: /6502 Peripherals/v1pa5 -> Net-(J72-Pad1)
- U10 pad 18: /6502 Peripherals/v1pa6 -> Net-(J73-Pad1)
- U10 pad 19: /6502 Peripherals/v1pa7 -> Net-(J74-Pad1)
- U10 pad 2: KBDAT -> Net-(J75-Pad1)
- U10 pad 3: /6502 Peripherals/v1pa8 -> Net-(J76-Pad1)
- U10 pad 6: KBCLK -> Net-(J77-Pad1)
- U10 pad 7: /6502 Peripherals/v1pa9 -> Net-(J78-Pad1)
- U11 pad 10: /6502 Peripherals/v2pb0 -> /6502 Peripherals 1/v3pb0
- U11 pad 11: /6502 Peripherals/v2pb1 -> /6502 Peripherals 1/v3pb1
- U11 pad 12: /6502 Peripherals/v2pb2 -> /6502 Peripherals 1/v3pb2
- U11 pad 13: /6502 Peripherals/v2pb3 -> /6502 Peripherals 1/v3pb3
- U11 pad 14: /6502 Peripherals/v2pb4 -> /6502 Peripherals 1/v3pb4
- U11 pad 15: /6502 Peripherals/v2pb5 -> /6502 Peripherals 1/v3pb5
- U11 pad 16: /6502 Peripherals/v2pb6 -> /6502 Peripherals 1/v3pb6
- U11 pad 17: /6502 Peripherals/v2pb7 -> /6502 Peripherals 1/v3pb7
- U11 pad 18: /6502 Peripherals/v2pb8 -> /6502 Peripherals 1/v3pb8
- U11 pad 19: /6502 Peripherals/v2pb9 -> /6502 Peripherals 1/v3pb9
- U11 pad 2: /6502 Peripherals/v2pa0 -> /6502 Peripherals 1/v3pa0
- U11 pad 21: ~V2IRQ -> ~V3IRQ
- U11 pad 23: ~IOCS -> Net-(J66-Pad1)
- U11 pad 24: a11 -> Net-(J65-Pad1)
- U11 pad 3: /6502 Peripherals/v2pa1 -> /6502 Peripherals 1/v3pa1
- U11 pad 39: /6502 Peripherals/v2pa9 -> /6502 Peripherals 1/v3pa9
- U11 pad 4: /6502 Peripherals/v2pa2 -> /6502 Peripherals 1/v3pa2
- U11 pad 40: /6502 Peripherals/v2pa8 -> /6502 Peripherals 1/v3pa8
- U11 pad 5: /6502 Peripherals/v2pa3 -> /6502 Peripherals 1/v3pa3
- U11 pad 6: /6502 Peripherals/v2pa4 -> /6502 Peripherals 1/v3pa4
- U11 pad 7: /6502 Peripherals/v2pa5 -> /6502 Peripherals 1/v3pa5
- U11 pad 8: /6502 Peripherals/v2pa6 -> /6502 Peripherals 1/v3pa6
- U11 pad 9: /6502 Peripherals/v2pa7 -> /6502 Peripherals 1/v3pa7
- U12 pad 10: /6502 Peripherals/v1pb0 -> v2pb0
- U12 pad 11: /6502 Peripherals/v1pb1 -> v2pb1
- U12 pad 12: /6502 Peripherals/v1pb2 -> v2pb2
- U12 pad 13: /6502 Peripherals/v1pb3 -> v2pb3
- U12 pad 14: /6502 Peripherals/v1pb4 -> v2pb4
- U12 pad 15: /6502 Peripherals/v1pb5 -> v2pb5
- U12 pad 16: /6502 Peripherals/v1pb6 -> v2pb6
- U12 pad 17: /6502 Peripherals/v1pb7 -> v2pb7
- U12 pad 18: Net-(U12-Pad18) -> v2pb8
- U12 pad 19: Net-(U12-Pad19) -> v2pb9
- U12 pad 2: /6502 Peripherals/v1pa0 -> v2pa0
- U12 pad 21: ~V1IRQ -> ~V2IRQ
- U12 pad 23: ~IOCS -> Net-(J50-Pad1)
- U12 pad 24: a12 -> Net-(J49-Pad1)
- U12 pad 3: /6502 Peripherals/v1pa1 -> v2pa1
- U12 pad 39: /6502 Peripherals/v1pa9 -> v2pa9
- U12 pad 4: /6502 Peripherals/v1pa2 -> v2pa2
- U12 pad 40: /6502 Peripherals/v1pa8 -> v2pa8
- U12 pad 5: /6502 Peripherals/v1pa3 -> v2pa3
- U12 pad 6: /6502 Peripherals/v1pa4 -> v2pa4
- U12 pad 7: /6502 Peripherals/v1pa5 -> v2pa5
- U12 pad 8: /6502 Peripherals/v1pa6 -> v2pa6
- U12 pad 9: /6502 Peripherals/v1pa7 -> v2pa7
- U3 pad 11: GND -> Net-(J30-Pad2)
- U3 pad 12: GND -> Net-(J31-Pad2)
- U3 pad 5: GND -> Net-(J25-Pad2)
- U3 pad 6: GND -> Net-(J24-Pad2)
- U3 pad 8: GND -> Net-(J27-Pad2)
- U3 pad 9: GND -> Net-(J28-Pad2)
- U5 pad 2: a10 -> Net-(J47-Pad2)
- U5 pad 3: ~IOCS -> Net-(J48-Pad2)
- U6 pad 11: ~RES -> Net-(J45-Pad1)
- U6 pad 14: Net-(D3-Pad1) -> Net-(D2-Pad1)
- U6 pad 15: Net-(D2-Pad1) -> Net-(D3-Pad1)
- U7 pad 2: Net-(R7-Pad1) -> /rdy
- U7 pad 36: +5V -> /be
- U7 pad 38: +5V -> /~so
- U7 pad 6: Net-(R8-Pad1) -> /~nmi
- U7 pad 7: Net-(U7-Pad7) -> /sync
- U8 pad 20: ~ROM_CS -> Net-(J21-Pad1)
- U8 pad 22: ~ROM_OE -> Net-(J20-Pad1)
- U8 pad 27: +5V -> Net-(J19-Pad1)
- U9 pad 20: ~RAM_CS -> Net-(J34-Pad1)
- U9 pad 22: ~RAM_CS -> Net-(J33-Pad1)
Routing:
- net 4Mhz_CLK: track 0.00 -> 319.9 mm, vias 0 -> 2
- net v1pa5: track 0.00 -> 234.1 mm, vias 0 -> 7
- net v1pa6: track 0.00 -> 224.1 mm, vias 0 -> 8
- net v1pa7: track 0.00 -> 219.3 mm, vias 0 -> 7
- net v1pb3: track 0.00 -> 199.0 mm, vias 0 -> 2
- net v1pb0: track 0.00 -> 196.6 mm, vias 0 -> 3
- net v1pb2: track 0.00 -> 191.0 mm, vias 0 -> 2
- net v1pb1: track 0.00 -> 181.2 mm, vias 0 -> 2
- net v1pb5: track 0.00 -> 161.3 mm, vias 0 -> 2
- net v1pb6: track 0.00 -> 158.9 mm, vias 0 -> 3
- net v1pb4: track 0.00 -> 157.9 mm, vias 0 -> 2
- net v1pb7: track 0.00 -> 157.3 mm, vias 0 -> 3
- net ~V3IRQ: track 0.00 -> 154.8 mm, vias 0 -> 3
- net a10: track 301.4 -> 149.2 mm, vias 6 -> 2
- net /6502 Peripherals/v1pa7: track 146.9 -> 0.00 mm
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Other:
- net class Default: via_dia 0.8 -> 0.6096; via_drill 0.4 -> 0.3048
- net class PWR: trace_width 0.2286 -> 0.3048; via_dia 0.8 -> 0.762; via_drill 0.4 -> 0.3048
- board text added: "+5V_UART"
- board text added: "/CTS"
- board text added: "/IRQX"
- board text added: "/NMI"
- board text added: "/RES"
- board text added: "/SO"
- board text added: "/WE"
- board text added: "10"
- board text added: "11"
- board text added: "12"
- board text added: "13"
- board text added: "1MHZ"
- board text added: "1MHz CPU Clock"
- board text added: "4"
- board text added: "4 BIT"
- board text added: "4MHZ"
- board text added: "4MHz Clock"
- board text added: "5"
- board text added: "5V"
- board text added: "6"
- board text added: "65C02 CPU"
- board text added: "76489 Audio"
- board text added: "8"
- board text added: "8 BIT"
- board text added: "8400-840F"
- board text added: "8800-880F"
- board text added: "9"
- board text added: "9000-900F"
- board text added: "A9"
- board text added: "Address Decoder 1"
- board text added: "Address Decoder 2"
- board text added: "Asynchronous Communication Interface Adapter 8200-820F"
- board text added: "Audio"
- board text added: "BE"
- board text added: "BLK"
- board text added: "Board revision: v002"
- board text added: "CPU Clock Selector"
- board text added: "EXT"
- board text added: "GRN"
- board text added: "IOCS"
- board text added: "IRQ"
- board text added: "Keyboard"
- board text added: "LCD"
- board text added: "LCD Physical Support"
- board text added: "LCD Selection"
- board text added: "PD0"
- board text added: "PD1"
- board text added: "PD2"
- board text added: "PD3"
- board text added: "PD4"
- board text added: "PD5"
- board text added: "PD6"
- board text added: "PIN12"
- board text added: "PIN13"
- board text added: "Port A"
- board text added: "Port B"
- board text added: "RAM_CE"
- board text added: "RAM_OE"
- board text added: "RDY"
- board text added: "ROM_CS"
- board text added: "ROM_OE"
- board text added: "ROM_WE"
- board text added: "Random Access Memory 32K 0000-7FFF"
- board text added: "Read Only Memory 24K A000-FFFF"
- board text added: "SYNC"
- board text added: "To CPU Clock Selector"
- board text added: "V2 Update: Tony Weil"
- board text added: "Versatile Interface Adapter #3"
- board text added: "https://github.com/tonylweil/db6502-V002"
- board text removed: "1MHz"
- board text removed: "1MHz System Clock"
- board text removed: "Address Bus"
- board text removed: "Address Decoder"
- board text removed: "Asynchronous Communication Interface Adapter"
- board text removed: "Board revision: v001"
- board text removed: "Central Processing Unit"
- board text removed: "Control Signals"
- board text removed: "Data Bus"
- board text removed: "External Clock Connector"
- board text removed: "Keyboard Connector PS/2"
- board text removed: "Random Access Memory"
- board text removed: "Read Only Memory"
- board text removed: "VIA 2 Port A"
- board text removed: "VIA 2 Port B"

Commit message: Update files to v002
Other:
- board text added: "Board revision: v002 5/10/2020"
- board text added: "https://github.com/tonylweil/6502"
- board text removed: "Board revision: v002"
- board text removed: "https://github.com/tonylweil/db6502-V002"

Commit message: Update files to v002
Parts:
- removed J36, J37: J, 65C02_Computer:PinHeader_1x02_P2.54mm_Vertical_Close
- removed J92: Jumper_NO_Small, 65C02_Computer:PinHeader_1x02_P2.54mm_Vertical_Close
- J35: value J -> CLK Jumper; footprint 65C02_Computer:PinHeader_1x02_P2.54mm_Vertical_Close -> 65C02_Computer:PinHeader_1x03_P2.54mm_Vertical_Close
- moved R14 25.8 mm to (54.6, 35.6), turned to 270 degrees
- moved C1 6.78 mm to (48.3, 23.5), turned to 180 degrees
- moved C3 6.75 mm to (88.9, 23.5), turned to 180 degrees
- moved J35 6.35 mm to (26.7, 43.2)
- moved J39 2.84 mm to (31.8, 26.7)
- moved J40 2.84 mm to (31.8, 29.2)
- moved J41 2.84 mm to (31.8, 31.8)
- moved J33 2.54 mm to (85.7, 83.8)
- moved J34 1.91 mm to (85.7, 86.4)
- moved R17 1.90 mm to (36.2, 23.5)
- moved C14 1.27 mm to (81.3, 83.8)
- moved J19 0.63 mm to (59.1, 83.8)
- moved J21 0.63 mm to (59.1, 88.9)
Routing:
- net 4Mhz_CLK: track 319.9 -> 0.00 mm, vias 2 -> 0
- net CLK: track 508.8 -> 441.2 mm, vias 7 -> 8
- net Net-(U14-Pad14): track 52.9 -> 29.6 mm
- net +5V: track 961.2 -> 983.6 mm, vias 12 -> 13
- net CLKOUT: track 20.3 -> 10.7 mm, vias 1 -> 0
- net GND: track 13.5 -> 19.8 mm, vias 2 -> 4
- net Net-(J22-Pad2): track 6.48 -> 10.5 mm
- net Net-(J32-Pad1): track 19.6 -> 15.9 mm, vias 1 -> 0
- net ~V2IRQ: track 226.9 -> 223.5 mm, vias 3 -> 4
- net Net-(J31-Pad2): track 19.2 -> 15.9 mm, vias 1 -> 0
- net Net-(J33-Pad1): track 26.9 -> 23.6 mm
- net Net-(J34-Pad1): track 28.5 -> 26.2 mm
- net ~ROM_OE: track 113.2 -> 111.9 mm
- net Net-(J19-Pad1): track 13.6 -> 12.2 mm
- net ~RAM_CS: track 76.4 -> 77.5 mm
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Other:
- board text added: "CLK IN"
- board text added: "CPU CLK"
- board text added: "CPU Clock"
- board text added: "External Clock Connector"
- board text added: "IRQX"
- board text removed: "/IRQX"
- board text removed: "1MHZ"
- board text removed: "1MHz CPU Clock"
- board text removed: "4MHZ"
- board text removed: "CPU Clock Selector"
- board text removed: "EXT"
- board text removed: "PIN12"
- board text removed: "PIN13"
- board text removed: "To CPU Clock Selector"

Commit message: Update files to v002
Routing:
- net Net-(J45-Pad2): track 62.1 -> 76.9 mm, vias 2 -> 3
- net GND: track 19.8 -> 13.9 mm, vias 4 -> 2
- net TxD: track 86.5 -> 91.9 mm, vias 3 -> 4
- net Net-(J45-Pad1): track 8.39 -> 12.7 mm
- net ~RTS: track 95.3 -> 99.3 mm, vias 3 -> 2
- net ~CTS: track 85.8 -> 89.1 mm
- net RxD: track 87.1 -> 89.4 mm, vias 4 -> 3
- net Net-(D3-Pad1): track 50.0 -> 51.3 mm
- net Net-(D2-Pad1): track 56.4 -> 57.1 mm
- net PUSBD+: vias 3 -> 2
